File: mechanical/KiCAD/OBD_PCB/TestProject_02.kicad_sch (KiCad schematic)
At the start: 45 parts, among them J1 USB_C_Receptacle_USB2.0_16P, J2 C-OBD-II-16M, J3 TXD_PAD, J4 RXD_PAD, U1 ESP32-C3-WROOM-02, U2 TPS54302, U3 USBLC6-2P6, U4 SN65HVD231

Commit message: Small layout changes, relocated the OBD PCB files to it's own folder. Final checks are needed.
Changed lines of the file:
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@@
 	(text "Switch to test\n3v3 power rail"
 		(exclude_from_sim no)
-		(at 112.268 164.084 0)
+		(at 117.602 163.83 0)
 		(effects
 			(font

Commit message: Touch ups, finalizing component placements
Parts:
- J2: footprint C-OBD-II-16M:COMTECH_C-OBD-II-16M -> custom_library:COMTECH_C-OBD-II-16M
Changed lines of the file:
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@@
 			)
 		)
-		(property "Footprint" "C-OBD-II-16M:COMTECH_C-OBD-II-16M"
+		(property "Footprint" "custom_library:COMTECH_C-OBD-II-16M"
 			(at 39.37 132.08 0)
 			(hide yes)

Commit message: Started the display PCB, since i use QSPI the current pinouts are not correct. Some ICs are still missing or not yet intergrated.
Parts:
- C4: value 100 nF -> 10 uF
- J2: footprint custom_library:COMTECH_C-OBD-II-16M -> C-OBD-II-16M:COMTECH_C-OBD-II-16M
Changed lines of the file:
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@@
 			)
 		)
-		(property "Footprint" "custom_library:COMTECH_C-OBD-II-16M"
+		(property "Footprint" "C-OBD-II-16M:COMTECH_C-OBD-II-16M"
 			(at 39.37 132.08 0)
 			(hide yes)
@@
 			)
 		)
-		(property "Value" "100 nF"
+		(property "Value" "10 uF"
 			(at 140.97 33.0199 0)
 			(show_name no)

Commit message: OBD and displa PCB are both basically finished, some files has to be generated and the PCBs can be ordered. Documentation should be the next step.
Parts:
- removed TEST_BTN1: SW_MEC_5E, Button_Switch_SMD:SW_SPST_EVQP2_MiddlePushTravel_H2.5mm, symbol Switch:SW_MEC_5E
- added JP2: Power Line Tester, Jumper:SolderJumper-2_P1.3mm_Open_Pad1.0x1.5mm, symbol Jumper:SolderJumper_2_Open
Connections:
- net +3.3V: now also JP2.2 (B)
- net at R8.2: now also JP2.1 (A)
Other:
- moved on the sheet: J3, J4, R8
Changed lines of the file:
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@@
 	)
 	(junction
+		(at 124.46 160.02)
+		(diameter 0)
+		(color 0 0 0 0)
+	)
+	(junction
 		(at 85.09 173.99)
 		(diameter 0)
@@
 	)
 	(junction
-		(at 124.46 160.02)
-		(diameter 0)
-		(color 0 0 0 0)
-	)
-	(junction
 		(at 85.09 189.23)
 		(diameter 0)
@@
 	(wire
 		(pts
-			(xy 125.73 172.72) (xy 124.46 172.72)
-		)
-		(stroke
-			(width 0)
-			(type default)
-		)
-	)
-	(wire
-		(pts
 			(xy 165.1 115.57) (xy 177.8 115.57)
 		)
@@
 	(wire
 		(pts
-			(xy 186.69 54.61) (xy 186.69 52.07)
-		)
-		(stroke
-			(width 0)
-			(type default)
-		)
-	)
-	(wire
-		(pts
 			(xy 26.67 171.45) (xy 26.67 175.26)
 		)
@@
 	(wire
 		(pts
-			(xy 124.46 160.02) (xy 124.46 170.18)
-		)
-		(stroke
-			(width 0)
-			(type default)
-		)
-	)
-	(wire
-		(pts
 			(xy 271.78 138.43) (xy 271.78 140.97)
 		)
@@
 	(wire
 		(pts
-			(xy 124.46 170.18) (xy 125.73 170.18)
-		)
-		(stroke
-			(width 0)
-			(type default)
-		)
-	)
-	(wire
-		(pts
 			(xy 66.04 91.44) (xy 66.04 96.52)
 		)
@@
 	(wire
 		(pts
-			(xy 124.46 172.72) (xy 124.46 175.26)
-		)
-		(stroke
-			(width 0)
-			(type default)
-		)
-	)
-	(wire
-		(pts
 			(xy 271.78 148.59) (xy 271.78 151.13)
 		)
@@
 	(wire
 		(pts
-			(xy 77.47 66.04) (xy 77.47 68.58)
+			(xy 124.46 160.02) (xy 134.62 160.02)
 		)
 		(stroke
@@
 	(wire
 		(pts
-			(xy 125.73 72.39) (xy 128.27 72.39)
+			(xy 77.47 66.04) (xy 77.47 68.58)
 		)
 		(stroke
@@
 	(wire
 		(pts
-			(xy 74.93 160.02) (xy 77.47 160.02)
+			(xy 125.73 72.39) (xy 128.27 72.39)
 		)
 		(stroke
@@
 	(wire
 		(pts
-			(xy 151.13 82.55) (xy 153.67 82.55)
+			(xy 74.93 160.02) (xy 77.47 160.02)
 		)
 		(stroke
@@
 	(wire
 		(pts
-			(xy 226.06 142.24) (xy 229.87 142.24)
+			(xy 151.13 82.55) (xy 153.67 82.55)
 		)
 		(stroke
@@
 	(wire
 		(pts
-			(xy 97.79 160.02) (xy 124.46 160.02)
+			(xy 226.06 142.24) (xy 229.87 142.24)
 		)
 		(stroke
@@
 	(wire
 		(pts
-			(xy 186.69 52.07) (xy 184.15 52.07)
+			(xy 184.15 52.07) (xy 196.85 52.07)
 		)
 		(stroke
@@
 	(wire
 		(pts
-			(xy 124.46 160.02) (xy 134.62 160.02)
+			(xy 97.79 160.02) (xy 124.46 160.02)
 		)
 		(stroke
@@
 	(wire
 		(pts
-			(xy 184.15 49.53) (xy 189.23 49.53)
+			(xy 184.15 49.53) (xy 196.85 49.53)
 		)
 		(stroke
@@
 	(wire
 		(pts
-			(xy 189.23 49.53) (xy 189.23 62.23)
-		)
-		(stroke
-			(width 0)
-			(type default)
-		)
-	)
-	(wire
-		(pts
 			(xy 256.54 138.43) (xy 259.08 138.43)
 		)
@@
 	(wire
 		(pts
-			(xy 135.89 170.18) (xy 135.89 172.72)
+			(xy 124.46 160.02) (xy 124.46 162.56)
 		)
 		(stroke
@@
 	(wire
 		(pts
+			(xy 124.46 172.72) (xy 124.46 175.26)
+		)
+		(stroke
+			(width 0)
+			(type default)
+		)
+	)
+	(wire
+		(pts
 			(xy 171.45 187.96) (xy 171.45 190.5)
 		)
@@
 	)
 	(symbol
-		(lib_id "Switch:SW_MEC_5E")
-		(at 130.81 172.72 0)
-		(unit 1)
-		(body_style 1)
-		(exclude_from_sim no)
-		(in_bom yes)
-		(on_board yes)
-		(in_pos_files yes)
-		(dnp no)
-		(fields_autoplaced yes)
-		(property "Reference" "TEST_BTN1"
-			(at 130.81 162.56 0)
-			(show_name no)
-			(do_not_autoplace no)
-			(effects
-				(font
-					(size 1.27 1.27)
-				)
-			)
-		)
-		(property "Value" "SW_MEC_5E"
-			(at 130.81 165.1 0)
-			(show_name no)
-			(do_not_autoplace no)
-			(effects
-				(font
-					(size 1.27 1.27)
-				)
-			)
-		)
-		(property "Footprint" "Button_Switch_SMD:SW_SPST_EVQP2_MiddlePushTravel_H2.5mm"
-			(at 130.81 165.1 0)
-			(hide yes)
-			(show_name no)
-			(do_not_autoplace no)
-			(effects
-				(font
-					(size 1.27 1.27)
-				)
-			)
-		)
-		(property "Datasheet" "https://www.apem.com/medias/download/MEC_switches_serie_MULTIMEC5E.pdf"
-			(at 130.81 165.1 0)
-			(hide yes)
-			(show_name no)
-			(do_not_autoplace no)
-			(effects
-				(font
-					(size 1.27 1.27)
-				)
-			)
-		)
-		(property "Description" "MEC 5E single pole normally-open tactile switch"
-			(at 130.81 172.72 0)
-			(hide yes)
-			(show_name no)
-			(do_not_autoplace no)
-			(effects
-				(font
-					(size 1.27 1.27)
-				)
-			)
-		)
-		(pin "2"
-		)
-		(pin "4"
-		)
-		(pin "1"
-		)
-		(pin "3"
-		)
-		(instances
-			(project "TestProject_02"
-				(path "/7255cca5-8951-4933-ab1b-c278e0bd5ab4"
-					(reference "TEST_BTN1")
-					(unit 1)
-				)
-			)
-		)
-	)
-	(symbol
 		(lib_id "power:GND")
 		(at 31.75 99.06 0)
@@
 	(symbol
 		(lib_id "Connector:Conn_01x01_Pin")
-		(at 186.69 59.69 90)
+		(at 201.93 52.07 0)
+		(mirror y)
 		(unit 1)
 		(body_style 1)
@@
 		(dnp no)
 		(property "Reference" "J4"
-			(at 189.484 55.88 90)
+			(at 198.12 53.594 90)
 			(show_name no)
 			(do_not_autoplace no)
@@
 		)
 		(property "Value" "RXD_PAD"
-			(at 189.484 58.42 90)
+			(at 200.66 53.594 90)
 			(show_name no)
 			(do_not_autoplace no)
@@
 		)
 		(property "Footprint" "TestPoint:TestPoint_Pad_2.0x2.0mm"
-			(at 186.69 59.69 0)
+			(at 201.93 52.07 0)
 			(hide yes)
 			(show_name no)
@@
 		)
 		(property "Datasheet" ""
-			(at 186.69 59.69 0)
+			(at 201.93 52.07 0)
 			(hide yes)
 			(show_name no)
@@
 		)
 		(property "Description" "Generic connector, single row, 01x01, script generated"
-			(at 186.69 59.69 0)
+			(at 201.93 52.07 0)
 			(hide yes)
 			(show_name no)
@@
 	(symbol
 		(lib_id "Connector:Conn_01x01_Pin")
-		(at 189.23 67.31 90)
+		(at 201.93 49.53 180)
 		(unit 1)
 		(body_style 1)
@@
 		(dnp no)
 		(property "Reference" "J3"
-			(at 189.992 63.5 90)
+			(at 198.12 46.99 90)
 			(show_name no)
 			(do_not_autoplace no)
@@
 		)
 		(property "Value" "TXD_PAD"
-			(at 189.992 66.04 90)
+			(at 200.66 46.99 90)
 			(show_name no)
 			(do_not_autoplace no)
@@
 		)
 		(property "Footprint" "TestPoint:TestPoint_Pad_2.0x2.0mm"
-			(at 189.23 67.31 0)
+			(at 201.93 49.53 0)
 			(hide yes)
 			(show_name no)
@@
 		)
 		(property "Datasheet" ""
-			(at 189.23 67.31 0)
+			(at 201.93 49.53 0)
 			(hide yes)
 			(show_name no)
@@
 		)
 		(property "Description" "Generic connector, single row, 01x01, script generated"
-			(at 189.23 67.31 0)
+			(at 201.93 49.53 0)
 			(hide yes)
 			(show_name no)
@@
 	)
 	(symbol
+		(lib_id "Jumper:SolderJumper_2_Open")
+		(at 124.46 167.64 90)
+		(unit 1)
+		(body_style 1)
+		(exclude_from_sim no)
+		(in_bom no)
+		(on_board yes)
+		(in_pos_files yes)
+		(dnp no)
+		(property "Reference" "JP2"
+			(at 127 166.3699 0)
+			(show_name no)
+			(do_not_autoplace no)
+			(effects
+				(font
+					(size 1.27 1.27)
+				)
+				(justify right)
+			)
+		)
+		(property "Value" "Power Line Tester"
+			(at 129.286 157.734 0)
+			(show_name no)
+			(do_not_autoplace no)
+			(effects
+				(font
+					(size 1.27 1.27)
+				)
+				(justify right)
+			)
+		)
+		(property "Footprint" "Jumper:SolderJumper-2_P1.3mm_Open_Pad1.0x1.5mm"
+			(at 124.46 167.64 0)
+			(hide yes)
+			(show_name no)
+			(do_not_autoplace no)
+			(effects
+				(font
+					(size 1.27 1.27)
+				)
+			)
+		)
+		(property "Datasheet" ""
+			(at 132.08 167.64 0)
+			(hide yes)
+			(show_name no)
+			(do_not_autoplace no)
+			(effects
+				(font
+					(size 1.27 1.27)
+				)
+			)
+		)
+		(property "Description" "Solder Jumper, 2-pole, open"
+			(at 129.54 167.64 0)
+			(hide yes)
+			(show_name no)
+			(do_not_autoplace no)
+			(effects
+				(font
+					(size 1.27 1.27)
+				)
+			)
+		)
+		(pin "2"
+		)
+		(pin "1"
+		)
+		(instances
+			(project "TestProject_02"
+				(path "/7255cca5-8951-4933-ab1b-c278e0bd5ab4"
+					(reference "JP2")
+					(unit 1)
+				)
+			)
+		)
+	)
+	(symbol
 		(lib_id "power:GND")
 		(at 271.78 156.21 0)
@@
 	(symbol
 		(lib_id "Device:R")
-		(at 124.46 179.07 180)
+		(at 124.46 179.07 0)
+		(mirror x)
 		(unit 1)
 		(body_style 1)
@@
 		(fields_autoplaced yes)
 		(property "Reference" "R8"
-			(at 127 177.7999 0)
+			(at 121.92 177.7999 0)
 			(show_name no)
 			(do_not_autoplace no)
@@
 		)
 		(property "Value" "1.5K"
-			(at 127 180.3399 0)
+			(at 121.92 180.3399 0)
 			(show_name no)
 			(do_not_autoplace no)
@@
 		)
 		(property "Footprint" "Resistor_SMD:R_0805_2012Metric"
-			(at 126.238 179.07 90)
+			(at 122.682 179.07 90)
 			(hide yes)
 			(show_name no)
@@
 	)
 	(symbol
+		(lib_name "SW_MEC_5E_1")
 		(lib_id "Switch:SW_MEC_5E")
 		(at 217.17 144.78 0)

Commit message: PCBs should be finished, they can be ordered. The plan was to finish the PCB design about a week ago. I already have the display and got two ESP devboard so i can start the software and test it.
Parts:
- C2, C3, C5: value 0.1 uF -> 100nF
- C4: value 10 uF -> 10uF
- R10, R11, R12, R13: footprint Resistor_SMD:R_0805_2012Metric -> Resistor_SMD:R_0603_1608Metric
Changed lines of the file:
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@@
 			)
 		)
-		(property "Value" "0.1 uF"
+		(property "Value" "100nF"
 			(at 157.48 33.0199 0)
 			(show_name no)
@@
 			)
 		)
-		(property "Footprint" "Resistor_SMD:R_0805_2012Metric"
+		(property "Footprint" "Resistor_SMD:R_0603_1608Metric"
 			(at 132.08 84.582 90)
 			(hide yes)
@@
 			)
 		)
-		(property "Footprint" "Resistor_SMD:R_0805_2012Metric"
+		(property "Footprint" "Resistor_SMD:R_0603_1608Metric"
 			(at 132.08 56.642 90)
 			(hide yes)
@@
 			)
 		)
-		(property "Value" "0.1 uF"
+		(property "Value" "100nF"
 			(at 71.12 157.4799 0)
 			(show_name no)
@@
 		(lib_id "Device:R")
 		(at 265.43 138.43 270)
-		(mirror x)
 		(unit 1)
 		(body_style 1)
@@
 			)
 		)
-		(property "Footprint" "Resistor_SMD:R_0805_2012Metric"
-			(at 265.43 140.208 90)
+		(property "Footprint" "Resistor_SMD:R_0603_1608Metric"
+			(at 265.43 136.652 90)
 			(hide yes)
 			(show_name no)
@@
 			)
 		)
-		(property "Footprint" "Resistor_SMD:R_0805_2012Metric"
+		(property "Footprint" "Resistor_SMD:R_0603_1608Metric"
 			(at 132.08 70.612 90)
 			(hide yes)
@@
 			)
 		)
-		(property "Value" "10 uF"
+		(property "Value" "10uF"
 			(at 140.97 33.0199 0)
 			(show_name no)
@@
 			)
 		)
-		(property "Value" "0.1 uF"
+		(property "Value" "100nF"
 			(at 275.59 146.0499 0)
 			(show_name no)

Commit message: Small changes due to via and silkscreen overlaps, moved every via-in-pad seperately from soldering pad. PCBs have been ordered. Some problems occured with the buttons since the ones i chose had a 5th mounting pin which was not present on the PCB. Also they asked about the button polarity and placement.Everything was corrected and the order moved to production.
Parts:
- BOOT2, EN1: LCSC (none) -> C713480
- C2, C3: LCSC (none) -> C1711
- C4, C7: LCSC (none) -> C32635
- C4A1: LCSC (none) -> C3039694
- C4B1, C5: LCSC (none) -> C1590
- C6A1, C6B1: LCSC (none) -> C29277
- C8: LCSC (none) -> C1621
- D1: LCSC (none) -> C78401
- D2: LCSC (none) -> C2480
- D3, D5: LCSC (none) -> C2297
- D4: LCSC (none) -> C10769
- D6: LCSC (none) -> C2293
- D7: LCSC (none) -> C2295
- D8: LCSC (none) -> C8678
- D9: LCSC (none) -> C14486
- F1: LCSC (none) -> C269104
- J1: LCSC (none) -> C165948
- J2, J3, J4: now left out of the parts list
- L1: LCSC (none) -> C84608
- R1, R3, R7: LCSC (none) -> C17414
- R10: LCSC (none) -> C22775
- R11, R12, R13: LCSC (none) -> C23138
- R2: LCSC (none) -> C17701
- R4, R5: LCSC (none) -> C27834
- R6: LCSC (none) -> C17514
- R8: LCSC (none) -> C4310
- U1: LCSC (none) -> C2934560
- U2: LCSC (none) -> C311983
- U3: LCSC (none) -> C2827693
- U4: LCSC (none) -> C129257
