File: mechanical/KiCAD/DISPLAY_PCB/display_pcb/display_pcb.kicad_pcb (KiCad board)
At the start: 4 copper layers, 49.9 x 56.4 mm, 50 parts, among them J1 USB_C_Receptacle_USB2.0_16P, J2 Conn_01x18_Socket, J3 Conn_01x01_Pin, J4 Conn_01x01_Pin, J5 Conn_01x02_Pin, Q1 AO3401A, U1 ESP32-S3-WROOM-1, U3 USBLC6-2P6, U4 TP4056-42-ESOP8, U5 TLV75733PDBV

Commit message: Módosítások a NYÁKon, volt egy hiba az útválasztó MOSFETtel, ezt csak a megrendelés után vettem észre és egy új NYÁK rendelést kellett indítani és lebeszélni JLCPCBvel hogy arra szereljék fel az alkatrészeket. A dokumentációk azok íródnak, a két dokumentáció az áramkörökről az készen van, maga a szakdolgozat dokumentuom az íródok.
Connections:
- Q1 pad 2: BTR + -> Net-(D8-K)
- Q1 pad 3: Net-(D8-K) -> BTR +
Routing:
- net Net-(D8-K): track 12.9 -> 15.0 mm
- net BTR +: track 43.6 -> 41.5 mm
Changed lines of the file:
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@@
 			(layers "F.Cu" "F.Mask" "F.Paste")
 			(roundrect_rratio 0.25)
-			(net "BTR +")
+			(net "Net-(D8-K)")
 			(pinfunction "S_2")
 			(pintype "passive")
@@
 			(layers "F.Cu" "F.Mask" "F.Paste")
 			(roundrect_rratio 0.25)
-			(net "Net-(D8-K)")
+			(net "BTR +")
 			(pinfunction "D_3")
 			(pintype "passive")
@@
 		(tags "SOT TO_SOT_SMD")
 		(property "Reference" "U5"
-			(at 0 -2.4 90)
+			(at -0.0085 2.499999 90)
 			(layer "F.SilkS")
 			(effects
@@
 			)
 		)
-		(attr exclude_from_pos_files exclude_from_bom)
+		(attr exclude_from_bom)
 		(duplicate_pad_numbers_are_jumpers no)
 		(fp_line
@@
 			)
 		)
-		(attr exclude_from_pos_files exclude_from_bom)
+		(attr exclude_from_bom)
 		(duplicate_pad_numbers_are_jumpers no)
 		(fp_line
@@
 	)
 	(segment
-		(start 98.8 83.9)
-		(end 97.2 83.9)
+		(start 121.850001 92.379)
+		(end 121.850001 95.204)
+		(width 0.5)
+		(layer "F.Cu")
+		(net "Net-(D8-K)")
+	)
+	(segment
+		(start 116.950001 92.304)
+		(end 117.846001 93.2)
+		(width 0.5)
+		(layer "F.Cu")
+		(net "Net-(D8-K)")
+	)
+	(segment
+		(start 123.750001 94.354)
+		(end 124.650001 95.254)
+		(width 0.5)
+		(layer "F.Cu")
+		(net "Net-(D8-K)")
+	)
+	(segment
+		(start 117.846001 93.2)
+		(end 121.029001 93.2)
+		(width 0.5)
+		(layer "F.Cu")
+		(net "Net-(D8-K)")
+	)
+	(segment
+		(start 124.500001 95.404)
+		(end 124.650001 95.254)
+		(width 0.5)
+		(layer "F.Cu")
+		(net "Net-(D8-K)")
+	)
+	(segment
+		(start 123.750001 92.379)
+		(end 123.750001 94.354)
+		(width 0.5)
+		(layer "F.Cu")
+		(net "Net-(D8-K)")
+	)
+	(segment
+		(start 121.650001 95.404)
+		(end 124.500001 95.404)
+		(width 0.5)
+		(layer "F.Cu")
+		(net "Net-(D8-K)")
+	)
+	(segment
+		(start 121.029001 93.2)
+		(end 121.850001 92.379)
+		(width 0.5)
+		(layer "F.Cu")
+		(net "Net-(D8-K)")
+	)
+	(segment
+		(start 121.850001 95.204)
+		(end 121.650001 95.404)
+		(width 0.5)
+		(layer "F.Cu")
+		(net "Net-(D8-K)")
+	)
+	(segment
+		(start 120.296 91.354)
+		(end 120.3 91.35)
 		(width 0.5)
 		(layer "F.Cu")
@@
 	)
 	(segment
-		(start 105.425 85.5)
-		(end 105.425 87.27)
+		(start 98.8 83.9)
+		(end 97.2 83.9)
 		(width 0.5)
 		(layer "F.Cu")
@@
 	)
 	(segment
-		(start 118.85 93.2)
-		(end 117.85 93.2)
+		(start 105.425 85.5)
+		(end 105.425 87.27)
 		(width 0.5)
 		(layer "F.Cu")
@@
 	)
 	(segment
-		(start 105.425 87.27)
-		(end 105.825 87.67)
+		(start 118.825001 91.354)
+		(end 120.296 91.354)
 		(width 0.5)
 		(layer "F.Cu")
@@
 	)
 	(segment
-		(start 117.85 93.2)
-		(end 116.95 92.3)
+		(start 105.425 87.27)
+		(end 105.825 87.67)
 		(width 0.5)
 		(layer "F.Cu")
@@
 	)
 	(via
-		(at 98.8 83.9)
+		(at 120.3 91.35)
 		(size 0.6)
 		(drill 0.3)
@@
 	)
 	(via
-		(at 105.425 83.9)
+		(at 98.8 83.9)
 		(size 0.6)
 		(drill 0.3)
@@
 	)
 	(via
-		(at 94.15 85.504)
+		(at 105.425 83.9)
 		(size 0.6)
 		(drill 0.3)
@@
 	)
 	(via
-		(at 118.85 93.2)
+		(at 94.15 85.504)
 		(size 0.6)
 		(drill 0.3)
@@
 	)
 	(segment
-		(start 105.425 83.9)
-		(end 105.45 83.9)
+		(start 120.3 89.9)
+		(end 118.85 88.45)
 		(width 0.5)
 		(layer "In2.Cu")
@@
 	)
 	(segment
-		(start 104.9 84.75)
-		(end 104.05 83.9)
+		(start 118.85 86.95)
+		(end 116.65 84.75)
 		(width 0.5)
 		(layer "In2.Cu")
@@
 	)
 	(segment
-		(start 116.65 84.75)
-		(end 104.9 84.75)
+		(start 118.85 88.45)
+		(end 118.85 86.95)
 		(width 0.5)
 		(layer "In2.Cu")
@@
 	)
 	(segment
-		(start 118.85 86.95)
-		(end 116.65 84.75)
+		(start 120.3 91.35)
+		(end 120.3 89.9)
 		(width 0.5)
 		(layer "In2.Cu")
@@
 	)
 	(segment
-		(start 94.846 85.504)
-		(end 96.45 83.9)
+		(start 105.425 83.9)
+		(end 105.45 83.9)
 		(width 0.5)
 		(layer "In2.Cu")
@@
 	)
 	(segment
-		(start 118.85 93.2)
-		(end 118.85 86.95)
+		(start 94.846 85.504)
+		(end 96.45 83.9)
 		(width 0.5)
 		(layer "In2.Cu")
@@
 	)
 	(segment
-		(start 98.8 83.9)
+		(start 104.9 84.75)
 		(end 104.05 83.9)
 		(width 0.5)
@@
 	)
 	(segment
-		(start 104.05 83.9)
-		(end 105.425 83.9)
+		(start 98.8 83.9)
+		(end 104.05 83.9)
 		(width 0.5)
 		(layer "In2.Cu")
@@
 	)
 	(segment
-		(start 121.850001 92.379)
-		(end 121.850001 95.204)
-		(width 0.5)
-		(layer "F.Cu")
-		(net "Net-(D8-K)")
-	)
-	(segment
-		(start 120.825001 91.354)
-		(end 121.850001 92.379)
-		(width 0.5)
-		(layer "F.Cu")
-		(net "Net-(D8-K)")
-	)
-	(segment
-		(start 118.825001 91.354)
-		(end 120.825001 91.354)
-		(width 0.5)
-		(layer "F.Cu")
-		(net "Net-(D8-K)")
-	)
-	(segment
-		(start 123.750001 94.354)
-		(end 124.650001 95.254)
-		(width 0.5)
-		(layer "F.Cu")
-		(net "Net-(D8-K)")
-	)
-	(segment
-		(start 124.500001 95.404)
-		(end 124.650001 95.254)
-		(width 0.5)
-		(layer "F.Cu")
-		(net "Net-(D8-K)")
-	)
-	(segment
-		(start 123.750001 92.379)
-		(end 123.750001 94.354)
-		(width 0.5)
-		(layer "F.Cu")
-		(net "Net-(D8-K)")
-	)
-	(segment
-		(start 121.650001 95.404)
-		(end 124.500001 95.404)
+		(start 116.65 84.75)
+		(end 104.9 84.75)
 		(width 0.5)
-		(layer "F.Cu")
-		(net "Net-(D8-K)")
+		(layer "In2.Cu")
+		(net "BTR +")
 	)
 	(segment
-		(start 121.850001 95.204)
-		(end 121.650001 95.404)
+		(start 104.05 83.9)
+		(end 105.425 83.9)
 		(width 0.5)
-		(layer "F.Cu")
-		(net "Net-(D8-K)")
+		(layer "In2.Cu")
+		(net "BTR +")
 	)
 	(segment
