File: mechanical/KiCAD/DISPLAY_PCB/display_pcb/display_pcb.kicad_sch (KiCad schematic)
At the start: 48 parts, among them J1 USB_C_Receptacle_USB2.0_16P, J2 Conn_01x18_Socket, J3 Conn_01x01_Pin, J4 Conn_01x01_Pin, J5 Conn_01x02_Pin, Q1 AO3401A, U1 ESP32-S3-WROOM-1, U3 USBLC6-2P6, U4 TP4056-42-ESOP8, U5 TLV75733PDBV

Commit message: Módosítások a NYÁKon, volt egy hiba az útválasztó MOSFETtel, ezt csak a megrendelés után vettem észre és egy új NYÁK rendelést kellett indítani és lebeszélni JLCPCBvel hogy arra szereljék fel az alkatrészeket. A dokumentációk azok íródnak, a két dokumentáció az áramkörökről az készen van, maga a szakdolgozat dokumentuom az íródok.
Connections:
- net BTR +: now also Q1.3 (D); no longer Q1.2 (S)
- net at C7.1, D8.1 (K), U5.1 (IN)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: now also Q1.2 (S); no longer Q1.3 (D)
